Commit message: 纠正了第三轴电机的力矩映射，link5吸盘质量略微补偿，link4加上了相机质量100g。在debug_node中添加了电机温度警报

File: src/arm2_task/urdf/arm2.urdf (robot description, URDF)
Before this commit: robot arm2.SLDASM, 6 links, 5 joints
Links:
- link Link_4: mass 0.0728159237766861 -> 0.172
- link Link_5: mass 0.337529561340392 -> 0.405
